File: USB_to_TTL/USB_to_TTL.kicad_sch (KiCad schematic)
At the start: 0 parts

Commit message: add cp2919
Parts:
- added C1, C2, C4: 0.1u, Capacitor_SMD:C_0603_1608Metric_Pad1.08x0.95mm_HandSolder, symbol Device:C_US
- added C3: 4.7u, Capacitor_SMD:C_0603_1608Metric_Pad1.08x0.95mm_HandSolder, symbol Device:C_US
- added D1: SP0503BAHT, Package_TO_SOT_SMD:SOT-143, symbol Power_Protection:SP0503BAHT
- added J1: USB_B, symbol Connector:USB_B
- added U1: CP2102N-Axx-xQFN28, Package_DFN_QFN:QFN-28-1EP_5x5mm_P0.5mm_EP3.35x3.35mm, symbol Interface_USB:CP2102N-Axx-xQFN28
Connections:
- new net: C3.2, C4.2, U1.6 (VDD)
- new net: U1.29 (GND), U1.3 (GND)
- new net D_+: D1.4 (K), J1.3 (D+), U1.4 (D+)
- new net D_-: D1.3 (K), J1.2 (D-), U1.5 (D-)
- new net GNDREF: C1.2, C2.2, C3.1, C4.1, D1.1 (A), J1.4 (GND), J1.5 (Shield)
- new net VBUS: C1.1, C2.1, D1.2 (K), J1.1 (VBUS), U1.7 (VREGIN), U1.8 (VBUS)

Commit message: 繼續作圖
Connections:
- net GNDREF: now also U1.29 (GND), U1.3 (GND)
- net RXD: now reaches U1.25 (RXD)
- net TXD: now reaches U1.26 (TXD)
- net VBUS renamed +5V
- no-connect marks 0 -> 19
Changed lines of the file:
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@@
+	)
+	(junction
+		(at 96.52 107.95)
+		(diameter 0)
+		(color 0 0 0 0)
 	)
 	(junction
@@
 		(color 0 0 0 0)
 	)
+	(junction
+		(at 123.19 15.24)
+		(diameter 0)
+		(color 0 0 0 0)
+	)
+	(no_connect
+		(at 109.22 97.79)
+	)
+	(no_connect
+		(at 109.22 72.39)
+	)
+	(no_connect
+		(at 109.22 74.93)
+	)
+	(no_connect
+		(at 109.22 57.15)
+	)
+	(no_connect
+		(at 109.22 85.09)
+	)
+	(no_connect
+		(at 109.22 87.63)
+	)
+	(no_connect
+		(at 109.22 77.47)
+	)
+	(no_connect
+		(at 109.22 67.31)
+	)
+	(no_connect
+		(at 109.22 80.01)
+	)
+	(no_connect
+		(at 109.22 92.71)
+	)
+	(no_connect
+		(at 109.22 95.25)
+	)
+	(no_connect
+		(at 109.22 82.55)
+	)
+	(no_connect
+		(at 109.22 54.61)
+	)
+	(no_connect
+		(at 109.22 46.99)
+	)
+	(no_connect
+		(at 109.22 64.77)
+	)
+	(no_connect
+		(at 109.22 52.07)
+	)
+	(no_connect
+		(at 109.22 59.69)
+	)
+	(no_connect
+		(at 83.82 41.91)
+	)
+	(no_connect
+		(at 109.22 49.53)
+	)
 	(wire
 		(pts
@@
 	(wire
 		(pts
+			(xy 96.52 107.95) (xy 146.05 107.95)
+		)
+		(stroke
+			(width 0)
+			(type default)
+		)
+	)
+	(wire
+		(pts
 			(xy 38.1 83.82) (xy 38.1 87.63)
 		)
@@
 	(wire
 		(pts
+			(xy 109.22 41.91) (xy 142.24 41.91)
+		)
+		(stroke
+			(width 0)
+			(type default)
+		)
+	)
+	(wire
+		(pts
 			(xy 29.21 87.63) (xy 35.56 87.63)
 		)
@@
 	(wire
 		(pts
+			(xy 109.22 44.45) (xy 142.24 44.45)
+		)
+		(stroke
+			(width 0)
+			(type default)
+		)
+	)
+	(wire
+		(pts
 			(xy 52.07 68.58) (xy 48.26 68.58)
 		)
@@
 	(wire
 		(pts
+			(xy 123.19 15.24) (xy 143.51 15.24)
+		)
+		(stroke
+			(width 0)
+			(type default)
+		)
+	)
+	(wire
+		(pts
 			(xy 74.93 15.24) (xy 93.98 15.24)
 		)
@@
 		(pts
 			(xy 35.56 87.63) (xy 38.1 87.63)
+		)
+		(stroke
+			(width 0)
+			(type default)
+		)
+	)
+	(wire
+		(pts
+			(xy 96.52 102.87) (xy 96.52 107.95)
 		)
 		(stroke
@@
 		)
 	)
+	(label "+5V"
+		(at 143.51 15.24 0)
+		(effects
+			(font
+				(size 1.27 1.27)
+			)
+			(justify left bottom)
+		)
+	)
+	(label "GND"
+		(at 146.05 107.95 0)
+		(effects
+			(font
+				(size 1.27 1.27)
+			)
+			(justify left bottom)
+		)
+	)
 	(label "D_+"
 		(at 45.72 73.66 0)
@@
 			)
 			(justify right bottom)
+		)
+	)
+	(label "RXD"
+		(at 142.24 44.45 0)
+		(effects
+			(font
+				(size 1.27 1.27)
+			)
+			(justify left bottom)
+		)
+	)
+	(label "TXD"
+		(at 142.24 41.91 0)
+		(effects
+			(font
+				(size 1.27 1.27)
+			)
+			(justify left bottom)
 		)
 	)
@@
 					(unit 1)
 				)
+			)
+		)
+	)
+	(symbol
+		(lib_id "power:GNDREF")
+		(at 96.52 107.95 0)
+		(unit 1)
+		(exclude_from_sim no)
+		(in_bom yes)
+		(on_board yes)
+		(dnp no)
+		(fields_autoplaced yes)
+		(property "Reference" "#PWR05"
+			(at 96.52 114.3 0)
+			(effects
+				(font
+					(size 1.27 1.27)
+				)
+				(hide yes)
+			)
+		)
+		(property "Value" "GNDREF"
+			(at 96.52 113.03 0)
+			(effects
+				(font
+					(size 1.27 1.27)
+				)
+			)
+		)
+		(property "Footprint" ""
+			(at 96.52 107.95 0)
+			(effects
+				(font
+					(size 1.27 1.27)
+				)
+				(hide yes)
+			)
+		)
+		(property "Datasheet" ""
+			(at 96.52 107.95 0)
+			(effects
+				(font
+					(size 1.27 1.27)
+				)
+				(hide yes)
+			)
+		)
+		(property "Description" "Power symbol creates a global label with name \"GNDREF\" , reference supply ground"
+			(at 96.52 107.95 0)
+			(effects
+				(font
+					(size 1.27 1.27)
+				)
+				(hide yes)
+			)
+		)
+		(pin "1"
+		)
+		(instances
+			(project "USB_to_TTL"
+				(path "/3709982b-ddb6-4217-a874-5034454930c8"
+					(reference "#PWR05")
+					(unit 1)
+				)

Commit message: 完成PCB佈線
Parts:
- added J2: Conn_01x04_Socket, Connector_PinSocket_2.54mm:PinSocket_1x04_P2.54mm_Vertical, symbol Connector:Conn_01x04_Socket
- J1: footprint (none) -> Connector_USB:USB_B_TE_5787834_Vertical
Connections:
- net +5V is gone; now on net VBUS: C1.1, C2.1, D1.2 (K), J1.1 (VBUS), U1.7 (VREGIN), U1.8 (VBUS)
- net GNDREF: now also J2.4 (Pin_4)
- net RXD: now also J2.2 (Pin_2)
- net TXD: now also J2.1 (Pin_1)
- net VBUS: now reaches C3.2, C4.2, U1.6 (VDD)
- net VBUS: now also J2.3 (Pin_3)
Changed lines of the file:
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@@
-	)
-	(junction
-		(at 35.56 87.63)
-		(diameter 0)
-		(color 0 0 0 0)
-	)
-	(junction
-		(at 96.52 107.95)
-		(diameter 0)
-		(color 0 0 0 0)
 	)
 	(junction
@@
 	)
 	(junction
+		(at 99.06 36.83)
+		(diameter 0)
+		(color 0 0 0 0)
+	)
+	(junction
 		(at 48.26 68.58)
 		(diameter 0)
@@
 	(wire
 		(pts
+			(xy 172.72 55.88) (xy 172.72 52.07)
+		)
+		(stroke
+			(width 0)
+			(type default)
+		)
+	)
+	(wire
+		(pts
 			(xy 110.49 15.24) (xy 123.19 15.24)
 		)
@@
 	(wire
 		(pts
-			(xy 96.52 107.95) (xy 146.05 107.95)
-		)
-		(stroke
-			(width 0)
-			(type default)
-		)
-	)
-	(wire
-		(pts
 			(xy 38.1 83.82) (xy 38.1 87.63)
 		)
@@
 	(wire
 		(pts
-			(xy 48.26 60.96) (xy 48.26 68.58)
+			(xy 172.72 52.07) (xy 175.26 52.07)
 		)
 		(stroke
@@
 	(wire
 		(pts
-			(xy 29.21 87.63) (xy 35.56 87.63)
+			(xy 99.06 36.83) (xy 111.76 36.83)
 		)
 		(stroke
@@
 			(width 0)
 			(type default)
+		)
+	)
+	(label "RXD"
+		(at 175.26 46.99 180)
+		(effects
+			(font
+				(size 1.27 1.27)
+			)
+			(justify right bottom)
 		)
 	)
@@
 		)
 	)
+	(label "VBUS"
+		(at 175.26 49.53 180)
+		(effects
+			(font
+				(size 1.27 1.27)
+			)
+			(justify right bottom)
+		)
+	)
 	(label "D_-"
 		(at 45.72 76.2 0)
@@
 		)
 	)
-	(label "+5V"
+	(label "VBUS"
 		(at 143.51 15.24 0)
-		(effects
-			(font
-				(size 1.27 1.27)
-			)
-			(justify left bottom)
-		)
-	)
-	(label "GND"
-		(at 146.05 107.95 0)
 		(effects
 			(font
@@
 		)
 	)
+	(label "TXD"
+		(at 175.26 44.45 180)
+		(effects
+			(font
+				(size 1.27 1.27)
+			)
+			(justify right bottom)
+		)
+	)
 	(label "RXD"
 		(at 142.24 44.45 0)
+		(effects
+			(font
+				(size 1.27 1.27)
+			)
+			(justify left bottom)
+		)
+	)
+	(label "VBUS"
+		(at 111.76 36.83 0)
 		(effects
 			(font
@@
 			)
 		)
-		(property "Footprint" ""
+		(property "Footprint" "Connector_USB:USB_B_TE_5787834_Vertical"
 			(at 41.91 74.93 0)
 			(effects
@@
 	(symbol
 		(lib_id "power:GNDREF")
+		(at 172.72 55.88 0)
+		(unit 1)
+		(exclude_from_sim no)
+		(in_bom yes)
+		(on_board yes)
+		(dnp no)
+		(property "Reference" "#PWR06"
+			(at 172.72 62.23 0)
+			(effects
+				(font
+					(size 1.27 1.27)
+				)
+				(hide yes)
+			)
+		)
+		(property "Value" "GNDREF"
+			(at 172.72 60.96 0)
+			(effects
+				(font
+					(size 1.27 1.27)
+				)
+			)
+		)
+		(property "Footprint" ""
+			(at 172.72 55.88 0)
+			(effects
+				(font
+					(size 1.27 1.27)
+				)
+				(hide yes)
+			)
+		)
+		(property "Datasheet" ""
+			(at 172.72 55.88 0)
+			(effects
+				(font
+					(size 1.27 1.27)
+				)
+				(hide yes)
+			)
+		)
+		(property "Description" "Power symbol creates a global label with name \"GNDREF\" , reference supply ground"
+			(at 172.72 55.88 0)
+			(effects
+				(font
+					(size 1.27 1.27)
+				)
+				(hide yes)
+			)
+		)
+		(pin "1"
+		)
+		(instances
+			(project "USB_to_TTL"
+				(path "/3709982b-ddb6-4217-a874-5034454930c8"
+					(reference "#PWR06")
+					(unit 1)
+				)
+			)
+		)
+	)
+	(symbol
+		(lib_id "power:GNDREF")
 		(at 134.62 31.75 0)
 		(unit 1)
@@
 	)
 	(symbol
-		(lib_id "power:PWR_FLAG")
-		(at 48.26 60.96 0)
-		(unit 1)
-		(exclude_from_sim no)
-		(in_bom yes)
-		(on_board yes)
-		(dnp no)
-		(fields_autoplaced yes)
-		(property "Reference" "#FLG01"
-			(at 48.26 59.055 0)
-			(effects
-				(font
-					(size 1.27 1.27)
-				)
-				(hide yes)
-			)
-		)
-		(property "Value" "PWR_FLAG"
-			(at 48.26 55.88 0)
-			(effects
-				(font
-					(size 1.27 1.27)
-				)
-			)
-		)
-		(property "Footprint" ""
-			(at 48.26 60.96 0)
-			(effects
-				(font
-					(size 1.27 1.27)
-				)
-				(hide yes)
-			)
-		)
-		(property "Datasheet" "~"
-			(at 48.26 60.96 0)
-			(effects
-				(font
-					(size 1.27 1.27)
-				)
-				(hide yes)
-			)
-		)
-		(property "Description" "Special symbol for telling ERC where power comes from"
-			(at 48.26 60.96 0)
-			(effects
-				(font
-					(size 1.27 1.27)
-				)
-				(hide yes)
-			)
-		)
-		(pin "1"
-		)
-		(instances
-			(project ""
-				(path "/3709982b-ddb6-4217-a874-5034454930c8"
-					(reference "#FLG01")
-					(unit 1)
-				)
-			)
-		)
-	)
-	(symbol
 		(lib_id "Device:C_US")
 		(at 99.06 29.21 0)
@@
 	)
 	(symbol
+		(lib_id "Connector:Conn_01x04_Socket")
+		(at 180.34 46.99 0)
+		(unit 1)
+		(exclude_from_sim no)
+		(in_bom yes)
+		(on_board yes)
+		(dnp no)
+		(fields_autoplaced yes)
+		(property "Reference" "J2"
+			(at 181.61 46.9899 0)
+			(effects
+				(font
+					(size 1.27 1.27)
+				)
+				(justify left)
+			)
+		)
+		(property "Value" "Conn_01x04_Socket"
+			(at 181.61 49.5299 0)
+			(effects
+				(font
+					(size 1.27 1.27)
+				)
+				(justify left)
+			)
+		)
+		(property "Footprint" "Connector_PinSocket_2.54mm:PinSocket_1x04_P2.54mm_Vertical"
+			(at 180.34 46.99 0)
+			(effects
+				(font
+					(size 1.27 1.27)
+				)
+				(hide yes)
+			)
+		)
+		(property "Datasheet" "~"
+			(at 180.34 46.99 0)
+			(effects
+				(font
+					(size 1.27 1.27)
+				)
+				(hide yes)
+			)
+		)
+		(property "Description" "Generic connector, single row, 01x04, script generated"
+			(at 180.34 46.99 0)
+			(effects
+				(font
+					(size 1.27 1.27)
+				)
+				(hide yes)
+			)
+		)
+		(pin "4"
+		)
+		(pin "3"
+		)
+		(pin "1"
+		)
+		(pin "2"
+		)
+		(instances
+			(project ""
+				(path "/3709982b-ddb6-4217-a874-5034454930c8"
+					(reference "J2")
+					(unit 1)
+				)
+			)
+		)
+	)
+	(symbol
 		(lib_id "power:GNDREF")
 		(at 38.1 91.44 0)
@@
 					(unit 1)
 				)
-			)
-		)
-	)
-	(symbol
-		(lib_id "power:PWR_FLAG")
-		(at 29.21 87.63 0)
-		(unit 1)
-		(exclude_from_sim no)
-		(in_bom yes)
-		(on_board yes)
-		(dnp no)
-		(fields_autoplaced yes)
-		(property "Reference" "#FLG02"
-			(at 29.21 85.725 0)
-			(effects
-				(font
-					(size 1.27 1.27)
-				)
-				(hide yes)
-			)
-		)
-		(property "Value" "PWR_FLAG"
-			(at 29.21 82.55 0)
-			(effects
-				(font
-					(size 1.27 1.27)
-				)
-			)
-		)
-		(property "Footprint" ""
-			(at 29.21 87.63 0)
-			(effects
-				(font
-					(size 1.27 1.27)
-				)
-				(hide yes)
-			)
-		)
-		(property "Datasheet" "~"
-			(at 29.21 87.63 0)
-			(effects
-				(font
-					(size 1.27 1.27)
-				)
-				(hide yes)
-			)
-		)
-		(property "Description" "Special symbol for telling ERC where power comes from"
-			(at 29.21 87.63 0)
-			(effects
-				(font
-					(size 1.27 1.27)
-				)
-				(hide yes)
-			)
-		)
-		(pin "1"
-		)
-		(instances
-			(project ""
-				(path "/3709982b-ddb6-4217-a874-5034454930c8"
-					(reference "#FLG02")
-					(unit 1)
-				)
