File: mouse_jiggler/mouse_jiggler.kicad_sch (KiCad schematic)
At the start: 0 parts

Commit message: 完成mouse jiggler
Parts:
- added SW1: CK_KMS2xxG, Button_Switch_SMD:SW_SPST_CK_KMS2xxGP, symbol Switch:CK_KMS2xxG
- added U1: Sparkfun_Pro_Micro, Arduino:Sparkfun_Pro_Micro, symbol arduino:Sparkfun_Pro_Micro
Connections:
- new net: SW1.2, U1.9 (~D6/A7)
- new net G: SW1.1, U1.23 (GND), U1.3 (GND), U1.4 (GND)
- no-connect marks 0 -> 22
